File: Projects/DTU Multimeter/KiCad/Multimeter/Multimeter.kicad_pcb (KiCad board)
At the start: 2 copper layers, 10 parts, among them U1 MCP3208-CI_P, U2 CD74HC4067E, U3 CD4053BE, U4 LM358P, U5 LM311N, U6 NE555P, U7 LM35DZ, U8 DS1307+

Commit message: Update DTU Multimeter PCB layout, schematic, and build guide
Add KiCad schematic fix scripts, ERC report, design plans,
and PlatformIO project configuration.
Parts:
- added BT1: CR2032, Battery:BatteryHolder_Keystone_3034_1x20mm, F.Cu at (675.0, 100.0)
- added BZ1: Piezo, Buzzer_Beeper:Buzzer_12x9.5RM7.6, F.Cu at (211.9, 25.5)
- added C1: 100n, Capacitor_THT:C_Disc_D5.0mm_W2.5mm_P2.50mm, F.Cu at (75.4, 20.2)
- added C2: 100n, Capacitor_THT:C_Disc_D5.0mm_W2.5mm_P2.50mm, F.Cu at (373.4, 140.8)
- added C3: 100n, Capacitor_THT:C_Disc_D5.0mm_W2.5mm_P2.50mm, F.Cu at (209.8, 99.0)
- added C4: 10u, Capacitor_THT:CP_Radial_D5.0mm_P2.50mm, F.Cu at (82.0, 21.5)
- added C5: 10u, Capacitor_THT:CP_Radial_D5.0mm_P2.50mm, F.Cu at (380.0, 144.5)
- added C6: 10u, Capacitor_THT:CP_Radial_D5.0mm_P2.50mm, F.Cu at (216.4, 105.2)
- added C7: 100n, Capacitor_THT:C_Disc_D5.0mm_W2.5mm_P2.50mm, F.Cu at (403.0, 238.0)
- added C8: 100n, Capacitor_THT:C_Disc_D5.0mm_W2.5mm_P2.50mm, F.Cu at (247.5, 88.5)
- added D1: Red, LED_THT:LED_D3.0mm, F.Cu at (127.2, 28.0)
- added D2: Green, LED_THT:LED_D3.0mm, F.Cu at (127.2, 33.5)
- added D3: Yellow, LED_THT:LED_D3.0mm, F.Cu at (127.2, 39.0)
- added D4: 1N4148, Diode_THT:D_DO-35_SOD27_P7.62mm_Horizontal, F.Cu at (199.9, 91.5)
- added F1: 10A, Fuse:Fuseholder_Clip-5x20mm_Keystone_3517_Inline_P23.11x6.76mm_D1.70mm_Horizontal, F.Cu at (29.4, 176.6)
- added F2: 500mA, Fuse:Fuseholder_Clip-5x20mm_Keystone_3517_Inline_P23.11x6.76mm_D1.70mm_Horizontal, F.Cu at (29.4, 184.5)
- added J1: Conn_01x01_Pin, Connector:Banana_Jack_1Pin, F.Cu at (46.5, 150.0)
- added J2: Conn_01x01_Pin, Connector:Banana_Jack_1Pin, F.Cu at (46.5, 162.6)
- added R1: 50.15, Resistor_THT:R_Axial_DIN0207_L6.3mm_D2.5mm_P10.16mm_Horizontal, F.Cu at (355.8, 92.8)
- added R10: 998, Resistor_THT:R_Axial_DIN0207_L6.3mm_D2.5mm_P10.16mm_Horizontal, F.Cu at (119.6, 94.5)
- added R11: 99.49, Resistor_THT:R_Axial_DIN0207_L6.3mm_D2.5mm_P10.16mm_Horizontal, F.Cu at (90.1, 100.6)
- added R12: 10.04, Resistor_THT:R_Axial_DIN0207_L6.3mm_D2.5mm_P10.16mm_Horizontal, F.Cu at (90.1, 96.5)
- added R13: 1.05, Resistor_THT:R_Axial_DIN0207_L6.3mm_D2.5mm_P10.16mm_Horizontal, F.Cu at (90.1, 92.5)
- added R14: 0.145, Resistor_THT:R_Axial_DIN0207_L6.3mm_D2.5mm_P10.16mm_Horizontal, F.Cu at (90.1, 88.5)
- added R15: 1.002M, Resistor_THT:R_Axial_DIN0207_L6.3mm_D2.5mm_P10.16mm_Horizontal, F.Cu at (20.1, 160.4)
- added R16: 100k, Resistor_THT:R_Axial_DIN0207_L6.3mm_D2.5mm_P10.16mm_Horizontal, F.Cu at (20.1, 164.5)
- added R17: 1.003M, Resistor_THT:R_Axial_DIN0207_L6.3mm_D2.5mm_P10.16mm_Horizontal, F.Cu at (247.3, 64.0)
- added R18: 10k, Resistor_THT:R_Axial_DIN0207_L6.3mm_D2.5mm_P10.16mm_Horizontal, F.Cu at (247.3, 68.0)
- added R19: 99.48, Resistor_THT:R_Axial_DIN0207_L6.3mm_D2.5mm_P10.16mm_Horizontal, F.Cu at (247.3, 72.0)
- added R2: 497, Resistor_THT:R_Axial_DIN0207_L6.3mm_D2.5mm_P10.16mm_Horizontal, F.Cu at (355.8, 96.9)
- added R20: 9.09k, Resistor_THT:R_Axial_DIN0207_L6.3mm_D2.5mm_P10.16mm_Horizontal, F.Cu at (214.3, 79.0)
- added R21: 1k, Resistor_THT:R_Axial_DIN0207_L6.3mm_D2.5mm_P10.16mm_Horizontal, F.Cu at (199.9, 83.0)
- added R22: 10k, Resistor_THT:R_Axial_DIN0207_L6.3mm_D2.5mm_P10.16mm_Horizontal, F.Cu at (402.9, 212.4)
- added R23: 10k, Resistor_THT:R_Axial_DIN0207_L6.3mm_D2.5mm_P10.16mm_Horizontal, F.Cu at (402.9, 216.5)
- added R24: 10k, Resistor_THT:R_Axial_DIN0207_L6.3mm_D2.5mm_P10.16mm_Horizontal, F.Cu at (402.9, 220.6)
- added R25: 330, Resistor_THT:R_Axial_DIN0207_L6.3mm_D2.5mm_P10.16mm_Horizontal, F.Cu at (106.8, 28.6)
- added R26: 330, Resistor_THT:R_Axial_DIN0207_L6.3mm_D2.5mm_P10.16mm_Horizontal, F.Cu at (106.8, 32.6)
- added R27: 330, Resistor_THT:R_Axial_DIN0207_L6.3mm_D2.5mm_P10.16mm_Horizontal, F.Cu at (106.8, 36.6)
- added R28: 10k, Resistor_THT:R_Axial_DIN0207_L6.3mm_D2.5mm_P10.16mm_Horizontal, F.Cu at (186.6, 22.9)
- added R29: 10k, Resistor_THT:R_Axial_DIN0207_L6.3mm_D2.5mm_P10.16mm_Horizontal, F.Cu at (182.5, 22.9)
- added R3: 4990, Resistor_THT:R_Axial_DIN0207_L6.3mm_D2.5mm_P10.16mm_Horizontal, F.Cu at (355.8, 101.0)
- added R4: 48.536k, Resistor_THT:R_Axial_DIN0207_L6.3mm_D2.5mm_P10.16mm_Horizontal, F.Cu at (355.8, 105.0)
- added R5: 498k, Resistor_THT:R_Axial_DIN0207_L6.3mm_D2.5mm_P10.16mm_Horizontal, F.Cu at (355.8, 109.0)
- added R6: 4.755M, Resistor_THT:R_Axial_DIN0207_L6.3mm_D2.5mm_P10.16mm_Horizontal, F.Cu at (355.8, 113.1)
- added R7: 10.06M, Resistor_THT:R_Axial_DIN0207_L6.3mm_D2.5mm_P10.16mm_Horizontal, F.Cu at (355.8, 117.2)
- added R8: 10.03M, Resistor_THT:R_Axial_DIN0207_L6.3mm_D2.5mm_P10.16mm_Horizontal, F.Cu at (355.8, 121.2)
- added R9: 10k, Resistor_THT:R_Axial_DIN0207_L6.3mm_D2.5mm_P10.16mm_Horizontal, F.Cu at (119.6, 98.5)
- added SW1: MODE, Button_Switch_THT:SW_PUSH_6mm, F.Cu at (324.4, 40.5)
- added SW2: FUNC, Button_Switch_THT:SW_PUSH_6mm, F.Cu at (332.9, 40.5)
- added SW3: RANGE, Button_Switch_THT:SW_PUSH_6mm, F.Cu at (341.5, 40.5)
- added SW4: SELECT, Button_Switch_THT:SW_PUSH_6mm, F.Cu at (350.1, 40.5)
- added Y1: 32.768kHz, Crystal:Crystal_C38-LF_D3.0mm_L8.0mm_Horizontal, F.Cu at (708.0, 94.2)
- moved U8 528.8 mm to (692.7, 87.2)
- moved U5 266.1 mm to (426.5, 235.7)
- moved A1 209.2 mm to (323.5, -37.9)
- moved U2 195.9 mm to (409.0, 149.7)
- moved U7 126.0 mm to (242.9, 22.0)
- moved DS1 116.9 mm to (182.8, 54.1)
- moved U1 106.9 mm to (249.8, 153.9)
- moved U4 93.1 mm to (219.5, 90.8)
- moved U6 90.1 mm to (266.0, 88.5)
- moved U3 45.4 mm to (100.5, 97.3)
Connections:
- A1 pad 22: unconnected-(A1-Pad22) -> /MUX_S0
- A1 pad 23: unconnected-(A1-Pad23) -> /MUX_S1
- A1 pad 24: unconnected-(A1-Pad24) -> /MUX_S2
- A1 pad 25: unconnected-(A1-Pad25) -> /MUX_S3
- A1 pad 26: unconnected-(A1-Pad26) -> /MUX_EN
- A1 pad 27: unconnected-(A1-Pad27) -> /CUR_A
- A1 pad 28: unconnected-(A1-Pad28) -> /CUR_B
- A1 pad 29: unconnected-(A1-Pad29) -> /CUR_C
- A1 pad 30: unconnected-(A1-Pad30) -> /CUR_INH
- A1 pad 31: unconnected-(A1-Pad31) -> /CAP_CHG
- A1 pad 32: unconnected-(A1-Pad32) -> /CAP_DIS
- A1 pad 33: unconnected-(A1-Pad33) -> /ISRC_EN
- A1 pad 50: unconnected-(A1-Pad50) -> /SPI_MISO
- A1 pad 51: unconnected-(A1-Pad51) -> /SPI_MOSI
- A1 pad 52: unconnected-(A1-Pad52) -> /SPI_SCK
- A1 pad 53: unconnected-(A1-Pad53) -> /SPI_CS
- A1 pad 5V_1: unconnected-(A1-+5V_1-Pad5V_1) -> VCC
- A1 pad AD10: unconnected-(A1-PadAD10) -> /LED_YEL
- A1 pad AD2: unconnected-(A1-PadAD2) -> /FREQ_IN
- A1 pad AD3: unconnected-(A1-PadAD3) -> /BTN_MODE
- A1 pad AD4: unconnected-(A1-PadAD4) -> /BTN_FUNC
- A1 pad AD5: unconnected-(A1-PadAD5) -> /BTN_RANGE
- A1 pad AD6: unconnected-(A1-PadAD6) -> /BTN_SEL
- A1 pad AD7: unconnected-(A1-PadAD7) -> /BUZZER
- A1 pad AD8: unconnected-(A1-PadAD8) -> /LED_RED
- A1 pad AD9: unconnected-(A1-PadAD9) -> /LED_GRN
- A1 pad GND2: unconnected-(A1-PadGND2) -> GND
- A1 pad SCL: unconnected-(A1-PadSCL) -> /I2C_SCL
- A1 pad SDA: unconnected-(A1-PadSDA) -> /I2C_SDA
- DS1 pad 1: unconnected-(DS1-VDD-Pad1) -> VCC
- DS1 pad 2: unconnected-(DS1-GND-Pad2) -> GND
- DS1 pad 3: unconnected-(DS1-SCK-Pad3) -> /I2C_SCL
- DS1 pad 4: unconnected-(DS1-SDA-Pad4) -> /I2C_SDA
- U1 pad 1: unconnected-(U1-CH0-Pad1) -> /MUX_COM
- U1 pad 10: unconnected-(U1-~CS/SHDN-Pad10) -> /SPI_CS
- U1 pad 11: unconnected-(U1-DIN-Pad11) -> /SPI_MOSI
- U1 pad 12: unconnected-(U1-DOUT-Pad12) -> /SPI_MISO
- U1 pad 13: unconnected-(U1-CLK-Pad13) -> /SPI_SCK
- U1 pad 14: unconnected-(U1-AGND-Pad14) -> GND
- U1 pad 15: unconnected-(U1-VREF-Pad15) -> VCC
- U1 pad 16: unconnected-(U1-VDD-Pad16) -> VCC
- U1 pad 2: unconnected-(U1-CH1-Pad2) -> /ADC_CH1
- U1 pad 3: unconnected-(U1-CH2-Pad3) -> /ADC_CH2
- U1 pad 4: unconnected-(U1-CH3-Pad4) -> /ADC_CH3
- U1 pad 5: unconnected-(U1-CH4-Pad5) -> /ADC_CH4
- U1 pad 6: unconnected-(U1-CH5-Pad6) -> /ADC_CH5
- U1 pad 9: unconnected-(U1-DGND-Pad9) -> GND
- U2 pad 1: unconnected-(U2-COM-Pad1) -> /MUX_COM
- U2 pad 10: unconnected-(U2-S0-Pad10) -> /MUX_S0
- U2 pad 11: unconnected-(U2-S1-Pad11) -> /MUX_S1
- U2 pad 12: unconnected-(U2-GND-Pad12) -> GND
- U2 pad 13: unconnected-(U2-S3-Pad13) -> /MUX_S3
- U2 pad 14: unconnected-(U2-S2-Pad14) -> /MUX_S2
- U2 pad 15: unconnected-(U2-~{E}-Pad15) -> /MUX_EN
- U2 pad 2: unconnected-(U2-I7-Pad2) -> Net-(U2-I7)
- U2 pad 24: unconnected-(U2-VCC-Pad24) -> VCC
- U2 pad 3: unconnected-(U2-I6-Pad3) -> Net-(U2-I6)
- U2 pad 4: unconnected-(U2-I5-Pad4) -> Net-(U2-I5)
- U2 pad 5: unconnected-(U2-I4-Pad5) -> Net-(U2-I4)
- U2 pad 6: unconnected-(U2-I3-Pad6) -> Net-(U2-I3)
- U2 pad 7: unconnected-(U2-I2-Pad7) -> Net-(U2-I2)
- U2 pad 8: unconnected-(U2-I1-Pad8) -> Net-(U2-I1)
- U2 pad 9: unconnected-(U2-I0-Pad9) -> Net-(U2-I0)
- U3 pad 1: unconnected-(U3-IN/OUT_BY-Pad1) -> Net-(U3-IN/OUT_BY)
- U3 pad 10: unconnected-(U3-B-Pad10) -> /CUR_B
- U3 pad 11: unconnected-(U3-A-Pad11) -> /CUR_A
- U3 pad 12: unconnected-(U3-AX_IN/OUT-Pad12) -> Net-(U3-AX_IN/OUT)
- U3 pad 13: unconnected-(U3-AY_IN/OUT-Pad13) -> Net-(U3-AY_IN/OUT)
- U3 pad 14: unconnected-(U3-OUT/IN_AX_OR_AY-Pad14) -> /SHUNT_NODE
- U3 pad 15: unconnected-(U3-OUT/IN_BX_OR_BY-Pad15) -> /SHUNT_NODE
- U3 pad 16: unconnected-(U3-VDD-Pad16) -> VCC
- U3 pad 2: unconnected-(U3-IN/OUT_BX-Pad2) -> Net-(U3-IN/OUT_BX)
- U3 pad 3: unconnected-(U3-IN/OUT_CY-Pad3) -> Net-(U3-IN/OUT_CY)
- U3 pad 4: unconnected-(U3-OUT/IN_CX_OR_CY-Pad4) -> /SHUNT_NODE
- U3 pad 5: unconnected-(U3-IN/OUT_CX-Pad5) -> Net-(U3-IN/OUT_CX)
- U3 pad 6: unconnected-(U3-INH-Pad6) -> /CUR_INH
- U3 pad 7: unconnected-(U3-VEE-Pad7) -> GND
- U3 pad 8: unconnected-(U3-VSS-Pad8) -> GND
- U3 pad 9: unconnected-(U3-C-Pad9) -> /CUR_C
- U4 pad 1: unconnected-(U4-Pad1) -> /ADC_CH3
- U4 pad 2: unconnected-(U4-Pad2) -> Net-(R20-Pad1)
- U4 pad 3: unconnected-(U4-Pad3) -> /SHUNT_NODE
- U4 pad 4: unconnected-(U4C-GND-Pad4) -> GND
- U4 pad 5: unconnected-(U4-Pad5) -> /ADC_CH2
- U4 pad 6: unconnected-(U4-Pad6) -> /ADC_CH4
- U4 pad 7: unconnected-(U4-Pad7) -> /ADC_CH4
- U4 pad 8: unconnected-(U4C-VCC-Pad8) -> VCC
- U5 pad 1: unconnected-(U5-GND-Pad1) -> GND
- U5 pad 2: unconnected-(U5-POS-Pad2) -> Net-(U5-POS)
- U5 pad 3: unconnected-(U5-NEG-Pad3) -> Net-(U5-NEG)
- U5 pad 4: unconnected-(U5-VCC--Pad4) -> GND
- U5 pad 7: unconnected-(U5-OUT-Pad7) -> /FREQ_IN
- U5 pad 8: unconnected-(U5-VCC+-Pad8) -> VCC
- U6 pad 1: unconnected-(U6-GND-Pad1) -> GND
- U6 pad 2: unconnected-(U6-TRIG-Pad2) -> /CAP_DIS
- U6 pad 3: unconnected-(U6-OUT-Pad3) -> /CAP_CHG
- U6 pad 4: unconnected-(U6-RESET-Pad4) -> /ISRC_EN
- U6 pad 5: unconnected-(U6-CONT-Pad5) -> Net-(U6-CONT)
- U6 pad 6: unconnected-(U6-THRES-Pad6) -> /CAP_DIS
- U6 pad 7: unconnected-(U6-DISCH-Pad7) -> Net-(U6-DISCH)
- U6 pad 8: unconnected-(U6-VCC-Pad8) -> VCC
- U7 pad 1: unconnected-(U7-+VS-Pad1) -> VCC
- U7 pad 2: unconnected-(U7-VOUT-Pad2) -> /ADC_CH5
- U7 pad 3: unconnected-(U7-GND-Pad3) -> GND
- U8 pad 1: unconnected-(U8-X1-Pad1) -> Net-(U8-X1)
- U8 pad 2: unconnected-(U8-X2-Pad2) -> Net-(U8-X2)
- U8 pad 3: unconnected-(U8-VBAT-Pad3) -> Net-(BT1-+)
- U8 pad 4: unconnected-(U8-GND-Pad4) -> GND
- U8 pad 5: unconnected-(U8-SDA-Pad5) -> /I2C_SDA
- U8 pad 6: unconnected-(U8-SCL-Pad6) -> /I2C_SCL
- U8 pad 8: unconnected-(U8-VCC-Pad8) -> VCC

Commit message: multimeter: snapshot full design before v1 simplification
Captures the current full-featured multimeter state:
- Complete schematic with all 22 measurement modes
- PCB placement with all ICs and passives
- Breadboard test firmware (voltage/resistance)
- Updated Mega footprint (proper headers + Z offset)
- New OLED footprint/symbol/3D model
- DTU single-sided PCB rules applied

This commit is the base for the full-version-multimeter branch.
Parts:
- removed DS1: OLED_128X64_1.3_I2C, OLED_128X64_1.3_I2C:LCD_OLED_128X64_1.3_I2C
- added U9: DM-OLED096-636, DM-OLED096-636:MODULE_DM-OLED096-636, F.Cu at (125.5, 51.5)
- F1, F2: footprint Fuse:Fuseholder_Clip-5x20mm_Keystone_3517_Inline_P23.11x6.76mm_D1.70mm_Horizontal -> Fuse:Fuseholder_Cylinder-5x20mm_Schurter_0031_8201_Horizontal_Open
- U2: footprint CD74HC4067E:DIP254P762X508-24 -> Package_DIP:DIP-24_18.0mmx34.29mm_W15.24mm
- moved Y1 600.3 mm to (108.0, 107.8), turned to 180 degrees
- moved U8 586.9 mm to (105.8, 94.2), turned to 90 degrees
- moved BT1 549.4 mm to (126.5, 131.0)
- moved U5 306.1 mm to (147.1, 110.6), turned to -90 degrees
- moved R22 303.7 mm to (120.5, 100.9)
- moved R23 303.7 mm to (120.5, 104.9)
- moved R24 303.7 mm to (120.5, 109.0)
- moved C7 275.9 mm to (156.9, 113.4)
- moved U2 264.1 mm to (152.0, 88.6), turned to 90 degrees
- moved C5 246.4 mm to (144.1, 73.4)
- moved C2 244.9 mm to (137.9, 73.4)
- moved F2 215.0 mm to (224.5, 94.2), turned to -90 degrees
- moved A1 214.1 mm to (154.5, 93.5)
- moved R8 207.3 mm to (150.5, 92.5), turned to -90 degrees
- moved R7 202.8 mm to (154.6, 92.5), turned to -90 degrees
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Connections:
- A1 pad 20: unconnected-(A1-Pad20) -> /I2C_SDA
- A1 pad 21: unconnected-(A1-Pad21) -> /I2C_SCL
- A1 pad SCL: /I2C_SCL -> unconnected-(A1-PadSCL)
- A1 pad SDA: /I2C_SDA -> unconnected-(A1-PadSDA)
Other:
- board outline added: 144 x 101 mm
