File: Projects/Class D Amplifier/hardware/kicad/sim/sim_a_vground.kicad_sch (KiCad schematic)
At the start: 6 parts, among them U1 TL074

Commit message: Class D amp: link the testbenches from the board sheet, both ways
The board schematic now carries a SIMULATION index in the free space below the
bridge: one clickable line per testbench, opening that testbench's project.
Each testbench carries a link back to the board.

These are hyperlinks, not hierarchical sheets, and that was not the first
choice - it is the result of trying the obvious thing and measuring what it
did. Attaching sim_b_triangle to classd.kicad_sch as a hierarchical sheet and
exporting the netlist showed three separate kinds of damage: the testbench's
12 V source welded straight onto the board's +12V rail, taking it from 23 pins
to 25; the sim's sources landing in the board netlist ready for Update PCB
from Schematic to push them onto copper; and worst, the sim sheet's U1, R4 and
R5 silently merging with the board parts of the same name, quietly rewiring
real components. A hierarchy is one electrical design, so anything inside it
is part of the board whether you meant it or not.

Getting the hyperlink right took measuring too. KiCad 10 refuses to load a
schematic where the link is spelled (hyperlink ...) as it is on the PCB, or
where it sits beside (uuid ...) rather than inside (effects ...). It also
rejects an href that is a bare relative path or a ${KIPRJMOD} variable, but
accepts a relative path carrying the file: scheme - which is what is used, so
the links survive the repository being checked out anywhere.

Also fixed while here: labels that sat beside a wire end rather than on it
left dangling endpoints, and the testbench supplies needed a ground PWR_FLAG
as well as a rail one. All four sheets now pass ERC with zero violations, and
the simulation checks still pass 16/16.
Other:
- note added: "<- back to the board schematic classd.kicad_pro"
Changed lines of the file:
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@@
+	(wire
+		(pts
+			(xy 17.78 43.18) (xy 27.94 43.18)
+		)
+		(stroke
+			(width 0)
+			(type default)
+		)
+	)
 	(wire
 		(pts
@@
 	(junction
 		(at 17.78 33.02)
+		(diameter 0)
+		(color 0 0 0 0)
+	)
+	(junction
+		(at 17.78 43.18)
 		(diameter 0)
 		(color 0 0 0 0)
@@
 		)
 	)
+	(text "<-  back to the board schematic   classd.kicad_pro"
+		(at 12.7 111.76 0)
+		(effects
+			(font
+				(size 1.6 1.6)
+			)
+			(justify left bottom)
+			(href "file:../classd.kicad_pro")
+		)
+	)
 	(symbol
 		(lib_id "Simulation_SPICE:VPULSE")
@@
 	)
 	(symbol
+		(lib_id "power:PWR_FLAG")
+		(at 27.94 43.18 0)
+		(unit 1)
+		(body_style 1)
+		(exclude_from_sim no)
+		(in_bom no)
+		(on_board no)
+		(in_pos_files no)
+		(dnp no)
+		(property "Reference" "#PWR004"
+			(at 30.734 41.91 0)
+			(hide yes)
+			(show_name no)
+			(do_not_autoplace no)
+			(effects
+				(font
+					(size 1.27 1.27)
+				)
+			)
+		)
+		(property "Value" "PWR_FLAG"
+			(at 30.734 44.45 0)
+			(show_name no)
+			(do_not_autoplace no)
+			(effects
+				(font
+					(size 1.27 1.27)
+				)
+			)
+		)
+		(property "Footprint" ""
+			(at 27.94 43.18 0)
+			(hide yes)
+			(show_name no)
+			(do_not_autoplace no)
+			(effects
+				(font
+					(size 1.27 1.27)
+				)
+			)
+		)
+		(property "Datasheet" ""
+			(at 27.94 43.18 0)
+			(hide yes)
+			(show_name no)
+			(do_not_autoplace no)
+			(effects
+				(font
+					(size 1.27 1.27)
+				)
+			)
+		)
+		(instances
+			(project "sim_a_vground"
+				(path "/a1000000-0000-4000-8000-000000000001"
+					(reference "#PWR004")
+					(unit 1)
+				)
+			)
+		)
+	)
+	(symbol
 		(lib_id "Device:R")
 		(at 45.72 30.48 0)
@@
 		(in_pos_files no)
 		(dnp no)
-		(property "Reference" "#PWR004"
+		(property "Reference" "#PWR005"
 			(at 48.26 20.32 0)
 			(hide yes)
@@
 			(project "sim_a_vground"
 				(path "/a1000000-0000-4000-8000-000000000001"
-					(reference "#PWR004")
+					(reference "#PWR005")
 					(unit 1)
 				)
@@
 		(in_pos_files no)
 		(dnp no)
-		(property "Reference" "#PWR005"
+		(property "Reference" "#PWR006"
 			(at 45.72 55.372 0)
 			(hide yes)
@@
 			(project "sim_a_vground"
 				(path "/a1000000-0000-4000-8000-000000000001"
-					(reference "#PWR005")
+					(reference "#PWR006")
 					(unit 1)
 				)
@@
 		(in_pos_files no)
 		(dnp no)
-		(property "Reference" "#PWR006"
+		(property "Reference" "#PWR007"
 			(at 60.96 55.372 0)
 			(hide yes)
@@
 			(project "sim_a_vground"
 				(path "/a1000000-0000-4000-8000-000000000001"
-					(reference "#PWR006")
+					(reference "#PWR007")
 					(unit 1)
 				)
@@
 		(in_pos_files no)
 		(dnp no)
-		(property "Reference" "#PWR007"
+		(property "Reference" "#PWR008"
 			(at 81.28 27.94 0)
 			(hide yes)
@@
 			(project "sim_a_vground"
 				(path "/a1000000-0000-4000-8000-000000000001"
-					(reference "#PWR007")
+					(reference "#PWR008")
 					(unit 1)
 				)
@@
 		(in_pos_files no)
 		(dnp no)
-		(property "Reference" "#PWR008"
+		(property "Reference" "#PWR009"
 			(at 81.788 53.34 0)
 			(hide yes)
@@
 			(project "sim_a_vground"
 				(path "/a1000000-0000-4000-8000-000000000001"
-					(reference "#PWR008")
+					(reference "#PWR009")
 					(unit 1)
 				)
@@
 		(in_pos_files no)
 		(dnp no)
-		(property "Reference" "#PWR009"
+		(property "Reference" "#PWR010"
 			(at 119.888 58.42 0)
 			(hide yes)
@@
 			(project "sim_a_vground"
 				(path "/a1000000-0000-4000-8000-000000000001"
-					(reference "#PWR009")
-					(unit 1)
-				)
+					(reference "#PWR010")
+					(unit 1)
+				)

Commit message: Class D amp: point the simulation links at the sheets, not the projects
Clicking a link opened the project manager and left you one click short of
the drawing. Windows resolves the two extensions to different programs:

  .kicad_pro -> kicad.exe     the project manager
  .kicad_sch -> eeschema.exe  the schematic editor, straight onto the sheet

So the board's index and the benches' back-links now name the .kicad_sch.
Eeschema still picks up the matching .kicad_pro sitting beside it, which is
what carries the netclass and the simulator workbook, so nothing is lost by
skipping the project manager.

Note for anyone setting this up on another machine: the association has to
point at the KiCad version the files were written with. On this PC
.kicad_sch resolved to the 9.0 eeschema while .kicad_pro resolved to 10.0,
and a 9.0 editor cannot open a 10.0 schematic.
Other:
- note added: "<- back to the board schematic classd.kicad_sch"
- note removed: "<- back to the board schematic classd.kicad_pro"
Changed lines of the file:
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@@
 		)
 	)
-	(text "<-  back to the board schematic   classd.kicad_pro"
+	(text "<-  back to the board schematic   classd.kicad_sch"
 		(at 12.7 111.76 0)
 		(effects
@@
 			)
 			(justify left bottom)
-			(href "file:../classd.kicad_pro")
+			(href "file:../classd.kicad_sch")
 		)
 	)
