File: Projects/Class D Amplifier/hardware/kicad/sim/sim_d_pwm.kicad_sch (KiCad schematic)
At the start: 8 parts, among them U1 LM311, U2 LM311

Commit message: Class D amp: link the testbenches from the board sheet, both ways
The board schematic now carries a SIMULATION index in the free space below the
bridge: one clickable line per testbench, opening that testbench's project.
Each testbench carries a link back to the board.

These are hyperlinks, not hierarchical sheets, and that was not the first
choice - it is the result of trying the obvious thing and measuring what it
did. Attaching sim_b_triangle to classd.kicad_sch as a hierarchical sheet and
exporting the netlist showed three separate kinds of damage: the testbench's
12 V source welded straight onto the board's +12V rail, taking it from 23 pins
to 25; the sim's sources landing in the board netlist ready for Update PCB
from Schematic to push them onto copper; and worst, the sim sheet's U1, R4 and
R5 silently merging with the board parts of the same name, quietly rewiring
real components. A hierarchy is one electrical design, so anything inside it
is part of the board whether you meant it or not.

Getting the hyperlink right took measuring too. KiCad 10 refuses to load a
schematic where the link is spelled (hyperlink ...) as it is on the PCB, or
where it sits beside (uuid ...) rather than inside (effects ...). It also
rejects an href that is a bare relative path or a ${KIPRJMOD} variable, but
accepts a relative path carrying the file: scheme - which is what is used, so
the links survive the repository being checked out anywhere.

Also fixed while here: labels that sat beside a wire end rather than on it
left dangling endpoints, and the testbench supplies needed a ground PWR_FLAG
as well as a rail one. All four sheets now pass ERC with zero violations, and
the simulation checks still pass 16/16.
Other:
- note added: "<- back to the board schematic classd.kicad_pro"
Changed lines of the file:
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@@
+	(wire
+		(pts
+			(xy 17.78 38.1) (xy 27.94 38.1)
+		)
+		(stroke
+			(width 0)
+			(type default)
+		)
+	)
 	(wire
 		(pts
@@
 	(junction
 		(at 17.78 27.94)
+		(diameter 0)
+		(color 0 0 0 0)
+	)
+	(junction
+		(at 17.78 38.1)
 		(diameter 0)
 		(color 0 0 0 0)
@@
 	)
 	(label "PWM_A"
-		(at 137.16 35.56 0)
+		(at 142.24 35.56 0)
 		(effects
 			(font
@@
 	)
 	(label "PWM_B"
-		(at 137.16 76.2 0)
+		(at 142.24 76.2 0)
 		(effects
 			(font
@@
 		)
 	)
+	(text "<-  back to the board schematic   classd.kicad_pro"
+		(at 12.7 111.76 0)
+		(effects
+			(font
+				(size 1.6 1.6)
+			)
+			(justify left bottom)
+			(href "file:../classd.kicad_pro")
+		)
+	)
 	(symbol
 		(lib_id "Simulation_SPICE:VDC")
@@
 	)
 	(symbol
+		(lib_id "power:PWR_FLAG")
+		(at 27.94 38.1 0)
+		(unit 1)
+		(body_style 1)
+		(exclude_from_sim no)
+		(in_bom no)
+		(on_board no)
+		(in_pos_files no)
+		(dnp no)
+		(property "Reference" "#PWR004"
+			(at 30.734 36.83 0)
+			(hide yes)
+			(show_name no)
+			(do_not_autoplace no)
+			(effects
+				(font
+					(size 1.27 1.27)
+				)
+			)
+		)
+		(property "Value" "PWR_FLAG"
+			(at 30.734 39.37 0)
+			(show_name no)
+			(do_not_autoplace no)
+			(effects
+				(font
+					(size 1.27 1.27)
+				)
+			)
+		)
+		(property "Footprint" ""
+			(at 27.94 38.1 0)
+			(hide yes)
+			(show_name no)
+			(do_not_autoplace no)
+			(effects
+				(font
+					(size 1.27 1.27)
+				)
+			)
+		)
+		(property "Datasheet" ""
+			(at 27.94 38.1 0)
+			(hide yes)
+			(show_name no)
+			(do_not_autoplace no)
+			(effects
+				(font
+					(size 1.27 1.27)
+				)
+			)
+		)
+		(instances
+			(project "sim_d_pwm"
+				(path "/a1000000-0000-4000-8000-000000000004"
+					(reference "#PWR004")
+					(unit 1)
+				)
+			)
+		)
+	)
+	(symbol
 		(lib_id "Simulation_SPICE:VPULSE")
 		(at 17.78 58.42 0)
@@
 		(in_pos_files no)
 		(dnp no)
-		(property "Reference" "#PWR004"
+		(property "Reference" "#PWR005"
 			(at 20.828 67.31 0)
 			(hide yes)
@@
 			(project "sim_d_pwm"
 				(path "/a1000000-0000-4000-8000-000000000004"
-					(reference "#PWR004")
+					(reference "#PWR005")
 					(unit 1)
 				)
@@
 		(in_pos_files no)
 		(dnp no)
-		(property "Reference" "#PWR005"
+		(property "Reference" "#PWR006"
 			(at 43.688 67.31 0)
 			(hide yes)
@@
 			(project "sim_d_pwm"
 				(path "/a1000000-0000-4000-8000-000000000004"
-					(reference "#PWR005")
+					(reference "#PWR006")
 					(unit 1)
 				)
@@
 		(in_pos_files no)
 		(dnp no)
-		(property "Reference" "#PWR006"
+		(property "Reference" "#PWR007"
 			(at 66.548 67.31 0)
 			(hide yes)
@@
 			(project "sim_d_pwm"
 				(path "/a1000000-0000-4000-8000-000000000004"
-					(reference "#PWR006")
+					(reference "#PWR007")
 					(unit 1)
 				)
@@
 		(in_pos_files no)
 		(dnp no)
-		(property "Reference" "#PWR007"
+		(property "Reference" "#PWR008"
 			(at 106.68 21.59 0)
 			(hide yes)
@@
 			(project "sim_d_pwm"
 				(path "/a1000000-0000-4000-8000-000000000004"
-					(reference "#PWR007")
+					(reference "#PWR008")
 					(unit 1)
 				)
@@
 		(in_pos_files no)
 		(dnp no)
-		(property "Reference" "#PWR008"
+		(property "Reference" "#PWR009"
 			(at 107.188 46.99 0)
 			(hide yes)
@@
 			(project "sim_d_pwm"
 				(path "/a1000000-0000-4000-8000-000000000004"
-					(reference "#PWR008")
+					(reference "#PWR009")
 					(unit 1)
 				)
@@
 		(in_pos_files no)
 		(dnp no)
-		(property "Reference" "#PWR009"
+		(property "Reference" "#PWR010"
 			(at 109.728 46.99 0)
 			(hide yes)
@@
 			(project "sim_d_pwm"
 				(path "/a1000000-0000-4000-8000-000000000004"
-					(reference "#PWR009")
+					(reference "#PWR010")
 					(unit 1)
 				)
@@
 		(in_pos_files no)
 		(dnp no)
-		(property "Reference" "#PWR010"
+		(property "Reference" "#PWR011"
 			(at 127 16.51 0)
 			(hide yes)
@@
 			(project "sim_d_pwm"
 				(path "/a1000000-0000-4000-8000-000000000004"
-					(reference "#PWR010")
+					(reference "#PWR011")
 					(unit 1)
 				)
@@
 		(in_pos_files no)
 		(dnp no)
-		(property "Reference" "#PWR011"
+		(property "Reference" "#PWR012"
 			(at 106.68 62.23 0)
 			(hide yes)
@@
 			(project "sim_d_pwm"
 				(path "/a1000000-0000-4000-8000-000000000004"
-					(reference "#PWR011")
+					(reference "#PWR012")
 					(unit 1)
 				)
@@
 		(in_pos_files no)
 		(dnp no)
-		(property "Reference" "#PWR012"
+		(property "Reference" "#PWR013"
 			(at 107.188 87.63 0)
 			(hide yes)
@@
 			(project "sim_d_pwm"
 				(path "/a1000000-0000-4000-8000-000000000004"
-					(reference "#PWR012")
+					(reference "#PWR013")
 					(unit 1)
 				)
@@
 		(in_pos_files no)
 		(dnp no)
-		(property "Reference" "#PWR013"
+		(property "Reference" "#PWR014"
 			(at 109.728 87.63 0)
 			(hide yes)
@@
 			(project "sim_d_pwm"
 				(path "/a1000000-0000-4000-8000-000000000004"
-					(reference "#PWR013")
+					(reference "#PWR014")
 					(unit 1)
 				)
@@
 		(in_pos_files no)
 		(dnp no)
-		(property "Reference" "#PWR014"
+		(property "Reference" "#PWR015"
 			(at 127 57.15 0)
 			(hide yes)
@@
 			(project "sim_d_pwm"
 				(path "/a1000000-0000-4000-8000-000000000004"
-					(reference "#PWR014")
-					(unit 1)
-				)
+					(reference "#PWR015")
+					(unit 1)
+				)

Commit message: Class D amp: point the simulation links at the sheets, not the projects
Clicking a link opened the project manager and left you one click short of
the drawing. Windows resolves the two extensions to different programs:

  .kicad_pro -> kicad.exe     the project manager
  .kicad_sch -> eeschema.exe  the schematic editor, straight onto the sheet

So the board's index and the benches' back-links now name the .kicad_sch.
Eeschema still picks up the matching .kicad_pro sitting beside it, which is
what carries the netclass and the simulator workbook, so nothing is lost by
skipping the project manager.

Note for anyone setting this up on another machine: the association has to
point at the KiCad version the files were written with. On this PC
.kicad_sch resolved to the 9.0 eeschema while .kicad_pro resolved to 10.0,
and a 9.0 editor cannot open a 10.0 schematic.
Other:
- note added: "<- back to the board schematic classd.kicad_sch"
- note removed: "<- back to the board schematic classd.kicad_pro"
Changed lines of the file:
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@@
 		)
 	)
-	(text "<-  back to the board schematic   classd.kicad_pro"
+	(text "<-  back to the board schematic   classd.kicad_sch"
 		(at 12.7 111.76 0)
 		(effects
@@
 			)
 			(justify left bottom)
-			(href "file:../classd.kicad_pro")
+			(href "file:../classd.kicad_sch")
 		)
 	)
