File: Projects/Class D Amplifier/hardware/kicad/sim/sim_e_driver.kicad_sch (KiCad schematic)
At the start: 25 parts, among them U20 CD4049UBE, U21 CD4049UBE, U22 CD4049UBE, U23 CD4049UBE, U6 HIP4082IPZ

Commit message: Class D amp: fold the bench-session findings back into the sheets
Every one of the seven testbenches has now been run in Eeschema's own
simulator and read back by hand, and the numbers match the harness: 214.6 kHz
carrier, 389 uV mirror error, 225 ns dead time, 11.6 W at fixed duty, and
13.0 W on the full chain with AUDIO_P bottoming out at exactly 4.00 V.

Three things that cost time during that session are now recorded on the
sheets themselves rather than being rediscovered:

- Measurements need a window. MAX over a whole run on E, F or G reads the
  t=0 initial-condition solve, where an uncharged bootstrap cap is a short
  and ties the switch node to the rail -- so G_AH appears to reach 12 V
  instead of its real 11.78 V. The E sheet now says so, with the FROM=/TO=
  form spelled out.
- A measurement takes a vector name, never an expression. KiCad binds each
  user-defined signal to user0, user1, ... and the sheets now ship with the
  useful expression already defined, so user0 exists as soon as you press Run:
  the mirror error on C, the differential output on F and G.
- On F and G, plot the difference rather than the two outputs. The whole
  filter is differential, nothing ties either output to ground, so the common
  mode is unfiltered and swings the full rail: each output measured to ground
  runs -3.8 V to +15.8 V while the load sees a clean 6.8 V. That is a property
  of the board, confirmed stable across a 20x change in timestep, and it is
  now written up in the build notes as an EMI consideration with the cost of
  the usual remedy measured (100 nF per output trims 1.6 V off the excursion
  and leaves the differential alone). No parts have been added.

The build notes also gain the common-mode section, and the sim README gains
the measured results and a short guide to driving KiCad's measurement panel.

Bench E's notes are wrapped short so they stay clear of the gate-load column,
which the longer text had been running through.
Other:
- note added: "Give every measurement a window. MAX over the whole run reads"
- note added: "MAX V(/G_AH) FROM=100u TO=150u reports the real 11.78 V."
- note added: "R23/R24 hold SW_A and SW_B near 0 V, standing in for the"
- note added: "The caps start empty and take ~50 us to fill, so read the dead"
- note added: "a volt below G_AL: the Schottky drop the high side runs on."
- note added: "charge -- the bridge itself is bench F."
- note added: "low-side FET being on. Without them the switch nodes float up"
- note added: "the t=0 solve, where the uncharged bootstrap cap is a short and"
- note added: "through the driver's own leakage and the bootstrap caps never"
- note added: "ties the switch node to the rail, so G_AH appears to reach 12 V."
- note added: "time from the far end of the run, not the start. Expect ~225 ns"
- note added: "with both outputs low at each commutation, and G_AH a quarter of"
- note removed: "Expect ~200 ns with both driver outputs low at every commutation, and G_AH about a quarter of a volt short of G_AL: that is the Schottky drop the high side runs on."
- note removed: "R23/R24 hold SW_A and SW_B near 0 V, standing in for the low-side FET being on. Leave them out and the switch nodes float up through the driver's own leakage until the bootstrap caps have barely a volt across them -- the bridge itself is bench F."
- note removed: "The bootstrap caps start empty and take ~50 us to reach 11.7 V, so read the dead time from the far end of the run, not the start."
Changed lines of the file:
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@@
 		)
 	)
-	(text "R23/R24 hold SW_A and SW_B near 0 V, standing in for the low-side FET being on. Leave them out and the switch nodes float up through the driver's own leakage until the bootstrap caps have barely a volt across them -- the bridge itself is bench F."
-		(at 12.7 223.52 0)
+	(text "R23/R24 hold SW_A and SW_B near 0 V, standing in for the"
+		(at 12.7 195.58 0)
 		(effects
 			(font
@@
 		)
 	)
-	(text "The bootstrap caps start empty and take ~50 us to reach 11.7 V, so read the dead time from the far end of the run, not the start."
-		(at 12.7 233.68 0)
+	(text "low-side FET being on. Without them the switch nodes float up"
+		(at 12.7 200.66 0)
 		(effects
 			(font
@@
 		)
 	)
-	(text "Expect ~200 ns with both driver outputs low at every commutation, and G_AH about a quarter of a volt short of G_AL: that is the Schottky drop the high side runs on."
-		(at 12.7 243.84 0)
+	(text "through the driver's own leakage and the bootstrap caps never"
+		(at 12.7 205.74 0)
+		(effects
+			(font
+				(size 1.27 1.27)
+			)
+			(justify left bottom)
+		)
+	)
+	(text "charge -- the bridge itself is bench F."
+		(at 12.7 210.82 0)
+		(effects
+			(font
+				(size 1.27 1.27)
+			)
+			(justify left bottom)
+		)
+	)
+	(text "The caps start empty and take ~50 us to fill, so read the dead"
+		(at 12.7 220.98 0)
+		(effects
+			(font
+				(size 1.27 1.27)
+			)
+			(justify left bottom)
+		)
+	)
+	(text "time from the far end of the run, not the start. Expect ~225 ns"
+		(at 12.7 226.06 0)
+		(effects
+			(font
+				(size 1.27 1.27)
+			)
+			(justify left bottom)
+		)
+	)
+	(text "with both outputs low at each commutation, and G_AH a quarter of"
+		(at 12.7 231.14 0)
+		(effects
+			(font
+				(size 1.27 1.27)
+			)
+			(justify left bottom)
+		)
+	)
+	(text "a volt below G_AL: the Schottky drop the high side runs on."
+		(at 12.7 236.22 0)
+		(effects
+			(font
+				(size 1.27 1.27)
+			)
+			(justify left bottom)
+		)
+	)
+	(text "Give every measurement a window. MAX over the whole run reads"
+		(at 12.7 246.38 0)
+		(effects
+			(font
+				(size 1.27 1.27)
+			)
+			(justify left bottom)
+		)
+	)
+	(text "the t=0 solve, where the uncharged bootstrap cap is a short and"
+		(at 12.7 251.46 0)
+		(effects
+			(font
+				(size 1.27 1.27)
+			)
+			(justify left bottom)
+		)
+	)
+	(text "ties the switch node to the rail, so G_AH appears to reach 12 V."
+		(at 12.7 256.54 0)
+		(effects
+			(font
+				(size 1.27 1.27)
+			)
+			(justify left bottom)
+		)
+	)
+	(text "MAX V(/G_AH) FROM=100u TO=150u reports the real 11.78 V."
+		(at 12.7 261.62 0)
 		(effects
 			(font
@@
 	)
 	(text ".tran 5n 150u uic"
-		(at 12.7 254 0)
+		(at 12.7 269.24 0)
 		(effects
 			(font
@@
 	)
 	(text "<-  back to the board schematic   classd.kicad_pro"
-		(at 12.7 269.24 0)
+		(at 12.7 279.4 0)
 		(effects
 			(font

Commit message: Class D amp: point the simulation links at the sheets, not the projects
Clicking a link opened the project manager and left you one click short of
the drawing. Windows resolves the two extensions to different programs:

  .kicad_pro -> kicad.exe     the project manager
  .kicad_sch -> eeschema.exe  the schematic editor, straight onto the sheet

So the board's index and the benches' back-links now name the .kicad_sch.
Eeschema still picks up the matching .kicad_pro sitting beside it, which is
what carries the netclass and the simulator workbook, so nothing is lost by
skipping the project manager.

Note for anyone setting this up on another machine: the association has to
point at the KiCad version the files were written with. On this PC
.kicad_sch resolved to the 9.0 eeschema while .kicad_pro resolved to 10.0,
and a 9.0 editor cannot open a 10.0 schematic.
Other:
- note added: "<- back to the board schematic classd.kicad_sch"
- note removed: "<- back to the board schematic classd.kicad_pro"
Changed lines of the file:
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@@
 		)
 	)
-	(text "<-  back to the board schematic   classd.kicad_pro"
+	(text "<-  back to the board schematic   classd.kicad_sch"
 		(at 12.7 279.4 0)
 		(effects
@@
 			)
 			(justify left bottom)
-			(href "file:../classd.kicad_pro")
+			(href "file:../classd.kicad_sch")
 		)
 	)
