File: Projects/Class D Amplifier/hardware/kicad/sim/sim_g_chain.kicad_sch (KiCad schematic)
At the start: 51 parts, among them Q1 IRF540N, Q2 IRF540N, Q3 IRF540N, Q4 IRF540N, U1 TL074, U2 TL074, U20 CD4049UBE, U21 CD4049UBE, U22 CD4049UBE, U23 CD4049UBE, U3 TL074, U4 LM311, U6 HIP4082IPZ, U7 LM311, U8 LM311

Commit message: Class D amp: fold the bench-session findings back into the sheets
Every one of the seven testbenches has now been run in Eeschema's own
simulator and read back by hand, and the numbers match the harness: 214.6 kHz
carrier, 389 uV mirror error, 225 ns dead time, 11.6 W at fixed duty, and
13.0 W on the full chain with AUDIO_P bottoming out at exactly 4.00 V.

Three things that cost time during that session are now recorded on the
sheets themselves rather than being rediscovered:

- Measurements need a window. MAX over a whole run on E, F or G reads the
  t=0 initial-condition solve, where an uncharged bootstrap cap is a short
  and ties the switch node to the rail -- so G_AH appears to reach 12 V
  instead of its real 11.78 V. The E sheet now says so, with the FROM=/TO=
  form spelled out.
- A measurement takes a vector name, never an expression. KiCad binds each
  user-defined signal to user0, user1, ... and the sheets now ship with the
  useful expression already defined, so user0 exists as soon as you press Run:
  the mirror error on C, the differential output on F and G.
- On F and G, plot the difference rather than the two outputs. The whole
  filter is differential, nothing ties either output to ground, so the common
  mode is unfiltered and swings the full rail: each output measured to ground
  runs -3.8 V to +15.8 V while the load sees a clean 6.8 V. That is a property
  of the board, confirmed stable across a 20x change in timestep, and it is
  now written up in the build notes as an EMI consideration with the cost of
  the usual remedy measured (100 nF per output trims 1.6 V off the excursion
  and leaves the differential alone). No parts have been added.

The build notes also gain the common-mode section, and the sim README gains
the measured results and a short guide to driving KiCad's measurement panel.

Bench E's notes are wrapped short so they stay clear of the gate-load column,
which the longer text had been running through.
Other:
- note added: "Measure over one audio cycle, past the bootstrap fill: RMS user0 FROM=400u TO=1400u gives 7.2 V, which is 13 W across 4 ohm, and MIN V(/AUDIO_P) FROM=400u TO=1400u gives 4.00 V. user0 is the differential output -- KiCad binds every user-defined signal to userN, and the measurement panel wants that name rather than the expression."
Changed lines of the file:
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@@
+		)
+	)
+	(text "Measure over one audio cycle, past the bootstrap fill: RMS user0 FROM=400u TO=1400u gives 7.2 V, which is 13 W across 4 ohm, and MIN V(/AUDIO_P) FROM=400u TO=1400u gives 4.00 V. user0 is the differential output -- KiCad binds every user-defined signal to userN, and the measurement panel wants that name rather than the expression."
+		(at 12.7 340.36 0)
+		(effects
+			(font
+				(size 1.27 1.27)
+			)
+			(justify left bottom)
 		)
 	)
 	(text ".tran 20n 1.4m uic"
-		(at 12.7 340.36 0)
+		(at 12.7 350.52 0)
 		(effects
 			(font
@@
 	)
 	(text "<-  back to the board schematic   classd.kicad_pro"
-		(at 12.7 350.52 0)
+		(at 12.7 360.68 0)
 		(effects
 			(font

Commit message: Class D amp: point the simulation links at the sheets, not the projects
Clicking a link opened the project manager and left you one click short of
the drawing. Windows resolves the two extensions to different programs:

  .kicad_pro -> kicad.exe     the project manager
  .kicad_sch -> eeschema.exe  the schematic editor, straight onto the sheet

So the board's index and the benches' back-links now name the .kicad_sch.
Eeschema still picks up the matching .kicad_pro sitting beside it, which is
what carries the netclass and the simulator workbook, so nothing is lost by
skipping the project manager.

Note for anyone setting this up on another machine: the association has to
point at the KiCad version the files were written with. On this PC
.kicad_sch resolved to the 9.0 eeschema while .kicad_pro resolved to 10.0,
and a 9.0 editor cannot open a 10.0 schematic.
Other:
- note added: "<- back to the board schematic classd.kicad_sch"
- note removed: "<- back to the board schematic classd.kicad_pro"
Changed lines of the file:
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@@
 		)
 	)
-	(text "<-  back to the board schematic   classd.kicad_pro"
+	(text "<-  back to the board schematic   classd.kicad_sch"
 		(at 12.7 360.68 0)
 		(effects
@@
 			)
 			(justify left bottom)
-			(href "file:../classd.kicad_pro")
+			(href "file:../classd.kicad_sch")
 		)
 	)
