File: Projects/BLE Digital Caliper/hardware/kicad/protoboard.kicad_sch (KiCad schematic)
At the start: 10 parts, among them J1 CALIPER, Q1 BC547, Q2 BC547, SW1 SEND, SW2 SEND+SP, U1 ESP32 DevKit

Commit message: BLE caliper: say which physical leg each transistor pin is
The schematic symbol numbers the BC547 C-B-E, so pin 1 is the collector
and, flat face toward you with the legs down, that is the left leg. The
drawing did not say so anywhere -- the symbol puts Base on the left and
stacks C and E on the right, so the pin numbers are the only thing
carrying it, and a reversed collector and emitter is the likeliest way to
build this wrong.

Both the sheet and level-shifter.md now carry the mapping and the meter
check that settles it independently: red probe on the middle leg, both
outer legs read about 0.7 V, and the higher of the two is the emitter
because the base-collector junction has the larger area and a lower drop
at the same test current. An hFE socket is definitive if the meter has
one.

Worth not trusting the table alone: datasheets differ on whether front
view means the flat face or the rounded one.
Other:
- note added: "A 2N3904 is the mirror image (E B C), so check"
- note added: "BC547: flat face toward you, legs down --"
- note added: "before soldering: diode mode, red on the middle"
- note added: "left = C = pin 1, middle = B = pin 2,"
- note added: "leg, both outer legs read ~0.7 V. The HIGHER of"
- note added: "right = E = pin 3."
- note added: "the two is the EMITTER."
- note removed: "A 2N3904 is E B C, the mirror image. If a stage"
- note removed: "BC547 pinout: flat face toward you, legs down,"
- note removed: "left to right = C B E."
- note removed: "will not switch, swap the outer two legs."
Changed lines of the file:
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@@
 		)
 	)
-	(text "BC547 pinout: flat face toward you, legs down,"
+	(text "BC547: flat face toward you, legs down --"
 		(at 10.16 133.35 0)
 		(effects
@@
 		)
 	)
-	(text "left to right = C  B  E."
+	(text "left = C = pin 1,  middle = B = pin 2,"
 		(at 10.16 137.16 0)
 		(effects
@@
 		)
 	)
-	(text "A 2N3904 is E  B  C, the mirror image. If a stage"
+	(text "right = E = pin 3."
 		(at 10.16 139.7 0)
 		(effects
@@
 		)
 	)
-	(text "will not switch, swap the outer two legs."
+	(text "A 2N3904 is the mirror image (E B C), so check"
 		(at 10.16 143.51 0)
 		(effects
 			(font
+				(size 1.5 1.5)
+			)
+			(justify left bottom)
+		)
+	)
+	(text "before soldering: diode mode, red on the middle"
+		(at 10.16 147.32 0)
+		(effects
+			(font
+				(size 1.5 1.5)
+			)
+			(justify left bottom)
+		)
+	)
+	(text "leg, both outer legs read ~0.7 V. The HIGHER of"
+		(at 10.16 149.86 0)
+		(effects
+			(font
+				(size 1.5 1.5)
+			)
+			(justify left bottom)
+		)
+	)
+	(text "the two is the EMITTER."
+		(at 10.16 152.4 0)
+		(effects
+			(font
