File: Projects/Vinyl ADC/hardware/kicad/vinyl_adc.kicad_sch (KiCad schematic)
At the start: 93 parts, among them J1 CLK SEL, J2 TO PI GPIO, J20 LINE IN L, J60 LINE IN R, U1 74HC244, U2 TL072, U20 TL074, U21 LM311, U3 74HCT132, U4 74HC4040, U5 74HC74, U6 74HC157, U60 TL074, U61 LM311, U7 74HC04, U8 74HC4049, X1 6.144MHz

Commit message: Vinyl ADC: split the board four ways so the mill can cut it
The one-board layout came out at 45 hand-soldered wire bridges, 17 vias and
25 ground pads the pour could not reach. The cause is one number: 2.54 mm DIP
pitch leaves 0.84 mm between pads, and a 1.0 mm track with 0.85 mm clearance
needs 2.7. Nothing passes between adjacent pins on this process, so every
connection goes round the outside of its package -- which makes routability a
function of space per part. The one-board version was 0.37 parts/cm2.

Three designs, four boards:

  common    power in, charge pump, +/-2.5 V reference, quantiser, DAC gates
  channel   one modulator: line in, three integrators, resonator, comparator
            -- ONE ARTWORK, MILLED TWICE
  digital   6.144 MHz clock, divider, interleave mux, level shift, Pi header

joined by three shrouded IDC ribbons. Odd pins are all ground, so every signal
has a grounded conductor either side of it in the cable; MCLK is why that
matters. Shrouded rather than bare strips because the rows carry supplies
against grounds and a reversed bare strip would put +5V across the ground
column.

Measured after routing: 42 wire bridges for a stereo set against 45 for one
board. The split did not halve the wire count -- what it bought is that every
ground pad now reaches its plane (25 stranded became 6), the boards build one
at a time, and two of the four are the same board. design-notes.md section 11
has the numbers and the two levers left untried.

New gate, tools/check_split.py: welds each ribbon's pin n to its partner's,
drops the connectors, and requires the resulting partition of every (ref, pin)
node to be identical to the one-page reference sheet's. It also proves channel
R is channel L with the refdes bumped by forty, which is what makes "one
artwork built twice" a checked claim. Sabotage-tested by moving the DAC gates
to the wrong board: it reports the severed nets, and nothing else does -- score,
ERC, geometry and footprint checks stay green on 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
Parts:
- C1: footprint (none) -> Capacitor_THT:CP_Radial_D10.0mm_P5.00mm
- C10, C11, C12, C13, C14, C15, C2, C21, C22, C23, C24, C25, C26, C27, C3, C61, C62, C63, C64, C65, C66, C67, C7, C8, C9: footprint (none) -> Capacitor_THT:C_Disc_D5.0mm_W2.5mm_P5.00mm
- C20, C60: footprint (none) -> Capacitor_THT:C_Rect_L11.0mm_W6.3mm_P10.00mm_MKT
- C4, C5, C6: footprint (none) -> Capacitor_THT:CP_Radial_D8.0mm_P3.50mm
- D1, D2: footprint (none) -> Diode_THT:D_DO-41_SOD81_P10.16mm_Horizontal
- J1: footprint (none) -> Connector_PinHeader_2.54mm:PinHeader_1x03_P2.54mm_Vertical
- J2: footprint (none) -> Connector_PinHeader_2.54mm:PinHeader_1x08_P2.54mm_Vertical
- J20, J60: footprint (none) -> TerminalBlock:TerminalBlock_bornier-2_P5.08mm
- R1, R2, R20, R21, R22, R23, R24, R25, R26, R27, R28, R29, R3, R30, R31, R32, R33, R34, R35, R36, R37, R4, R5, R60, R61, R62, R63, R64, R65, R66, R67, R68, R69, R70, R71, R72, R73, R74, R75, R76, R77: footprint (none) -> Resistor_THT:R_Axial_DIN0207_L6.3mm_D2.5mm_P7.62mm_Horizontal
- RV20, RV60: footprint (none) -> Potentiometer_THT:Potentiometer_Bourns_3296W_Vertical
- U1: footprint (none) -> Package_DIP:DIP-20_W7.62mm_LongPads
- U2, U21, U61, X1: footprint (none) -> Package_DIP:DIP-8_W7.62mm_LongPads
- U20, U3, U5, U60, U7: footprint (none) -> Package_DIP:DIP-14_W7.62mm_LongPads
- U4, U6, U8: footprint (none) -> Package_DIP:DIP-16_W7.62mm_LongPads
