File: Projects/Vinyl ADC/hardware/kicad/reference/vinyl_adc.kicad_sch (KiCad schematic)
At the start: 93 parts, among them J1 CLK SEL, J2 TO PI GPIO, J20 LINE IN L, J60 LINE IN R, U1 74HC244, U2 TL072, U20 TL074, U21 LM311, U3 74HCT132, U4 74HC4040, U5 74HC74, U6 74HC157, U60 TL074, U61 LM311, U7 74HC04, U8 74HC4049, X1 6.144MHz

Commit message: Vinyl ADC: rebuild as three stacking boards
The four-board split fixed the ground plane and not the congestion --
45 wire bridges became 42, and the bridge count barely moved however the
blocks were arranged. So this moves the cut lines rather than adding more
boards.

Each channel board now carries its own 74HC74 and 74HC04, so the modulator
loop closes on one board instead of crossing a ribbon. Measured on the old
common board, 59 of its 84 F.Cu segments were per-channel CMP/DAC/Q traffic;
that is what leaves with them. The TL074 becomes two TL072s per channel, so
the integrator pairs can sit apart instead of seventeen resistors competing
for one package's perimeter. What remains of the common board is power and
the reference, so it is now vinyl_adc_power.

The five IDC ribbons become one 2x8 stacking bus -- same pinout, same
coordinates on every board, 11 mm standoffs. ONE position, not a socket and
a header side by side: a middle board has to present a socket upwards and
pins downwards at the same XY, and two separate parts cannot do that on a
single-sided board. Both channel boards are still one artwork, so nothing on
the copper may name a channel: the flip-flop drives a neutral Q_OUT and a
shunt maps it to QL or QR.

Boards are 100x100 with four M3 holes and the bus locked on the centreline,
ground row outermost so the signals open into the board rather than the edge.
pcb_fixture.py stamps that geometry; check_fixture.py proves the three
artworks still agree, testing pad position AND pin number -- a board left
un-rotated still bolts onto the standoffs and puts +5V across the ground
column.

Every project gets its own directory. KiCad resolves fp-lib-table, the
session state and ${KIPRJMOD} from the project folder, so five projects
sharing one directory made them fight over it.

pcb_link.py stamps each footprint with its schematic symbol UUID.
pcb_build.py never wrote them, so cross-probing had never worked on this
project at all -- the board is otherwise valid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
Parts:
- removed C12, C14: 100n, Capacitor_THT:C_Disc_D5.0mm_W2.5mm_P5.00mm, symbol Device:C
- removed U20, U60: TL074, Package_DIP:DIP-14_W7.62mm_LongPads, symbol Amplifier_Operational:TL074
- removed U5: 74HC74, Package_DIP:DIP-14_W7.62mm_LongPads, symbol 74xx:74HC74
- removed U7: 74HC04, Package_DIP:DIP-14_W7.62mm_LongPads, symbol 74xx:74HC04
- added C28, C29, C30, C31, C68, C69, C70, C71: 100n, Capacitor_THT:C_Disc_D5.0mm_W2.5mm_P5.00mm, symbol Device:C
- added U20, U22, U60, U62: TL072, Package_DIP:DIP-8_W7.62mm_LongPads, symbol Amplifier_Operational:TL072
- added U23, U63: 74HC74, Package_DIP:DIP-14_W7.62mm_LongPads, symbol 74xx:74HC74
- added U24, U64: 74HC04, Package_DIP:DIP-14_W7.62mm_LongPads, symbol 74xx:74HC04
- RV20, RV60: footprint Potentiometer_THT:Potentiometer_Bourns_3296W_Vertical -> Connector_PinHeader_2.54mm:PinHeader_1x03_P2.54mm_Horizontal
Connections:
- net +5V: now also C28.1, C30.1, C31.1, C68.1, C70.1, C71.1, U20.8 (V+), U22.8 (V+), U23.1 (~{R}), U23.10 (~{S}), U23.13 (~{R}), U23.14 (VCC), U23.4 (~{S}), U24.14 (VCC), U60.8 (V+), U62.8 (V+), U63.1 (~{R}), U63.10 (~{S}), U63.13 (~{R}), U63.14 (VCC), U63.4 (~{S}), U64.14 (VCC)
- net -5V: now also C29.2, C69.2, U20.4 (V-), U22.4 (V-), U60.4 (V-), U62.4 (V-)
- net CMP_L: now also U23.2 (D)
- net CMP_R: now also U63.2 (D)
- net DACN_L: now also U24.2
- net DACN_R: now also U64.2
- net DACP_L: now also U24.4
- net DACP_R: now also U64.4
- net GND: now also C28.2, C29.1, C30.2, C31.2, C68.2, C69.1, C70.2, C71.2, U20.3 (+), U20.5 (+), U22.3 (+), U22.5 (+), U23.11 (C), U23.12 (D), U23.7 (GND), U24.11, U24.13, U24.5, U24.7 (GND), U24.9, U60.3 (+), U60.5 (+), U62.3 (+), U62.5 (+), U63.11 (C), U63.12 (D), U63.7 (GND), U64.11, U64.13, U64.5, U64.7 (GND), U64.9
- net MCLK: now also U23.3 (C), U63.3 (C)
- net QL: now also U23.5 (Q), U24.1
- net QNL: now also U23.6 (~{Q}), U24.3
- net QNR: now also U63.6 (~{Q}), U64.3
- net QR: now also U63.5 (Q), U64.1
- net at C64.1, R68.2, R69.2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: now also U62.2 (-)
- net at C63.1, R64.2, R65.2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: now also U60.6 (-)
- net at C63.2, R68.1: now also U60.7
- net at C64.2, R71.1, R73.1: now also U62.1
- net at C23.2, R28.1: now also U20.7
- net at C24.1, R28.2, R29.2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: now also U22.2 (-)
- net at C22.2, R24.1: now also U20.1
- net at C23.1, R24.2, R25.2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: now also U20.6 (-)
- net at C24.2, R31.1, R33.1: now also U22.1
- net at R27.1, R32.2: now also U22.7
- net at R71.2, R72.1: now also U62.6 (-)
- net at C62.1, R61.2, R62.2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: now also U60.2 (-)
- net at R67.1, R72.2: now also U62.7
- net at R31.2, R32.1: now also U22.6 (-)
- net at C22.1, R21.2, R22.2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: now also U20.2 (-)
- net at C62.2, R64.1: now also U60.1
- no-connect marks 20 -> 30
