File: Projects/Class D Amplifier/hardware/kicad/classd.refined.kicad_pcb (KiCad board)
At the start: 2 copper layers, 186.4 x 104 mm, 61 parts, among them J1 PWR IN 12V, J2 LINE IN, J3 SPEAKER 4R, Q1 IRF540N, Q2 IRF540N, Q3 IRF540N, Q4 IRF540N, U1 TL074, U2 LM311, U3 LM311, U4 LM311, U5 CD4049UBE, U6 HIP4082IPZ

Commit message: Class D: the autoplace and routing experiments, hand and machine
Both placements of the same board, each carried through refine and route, plus
the DRC dump and the Freerouting session files.

Measured on these files with the same router pass and the same cnc clearance
profile: the hand placement needs 17 hand-soldered links against the machine
placement's 26, while beating it on normalised wirelength as well, 0.1053 to
0.1184. Worth keeping the pair around -- one netlist with two placements is the
only way to compare a placer against anything.
Parts:
- moved R18 23.0 mm to (196.1, 105.8)
- moved R20 23.0 mm to (164.6, 105.7)
- moved R19 23.0 mm to (196.1, 119.4)
- moved R21 23.0 mm to (172.2, 119.4)
- moved C1 23.0 mm to (77.6, 57.9)
- moved C4 23.0 mm to (180.4, 114.1)
- moved L2 23.0 mm to (165.5, 88.1)
- moved TP5 23.0 mm to (211.1, 91.5)
- moved C14 23.0 mm to (167.6, 40.7)
- moved J1 23.0 mm to (102.8, 38.6)
- moved J2 23.0 mm to (145.0, 38.6)
- moved J3 23.0 mm to (184.7, 38.6)
- moved L1 23.0 mm to (200.3, 59.9)
- moved R22 23.0 mm to (198.2, 47.8)
- moved C13 23.0 mm to (190.4, 55.7)
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Routing:
- added copper zone on B.Cu, net GND
- removed copper zone on F.Cu, net GND
Other:
- board size 186.4 x 104 mm -> 190.5 x 104 mm
- board text added: "SRM-20 stroke 203.2 x 152.4"
- board text added: "via blank 190 x 140"
