File: Projects/Class D Amplifier/hardware/kicad/classd.refined.routed.kicad_pcb (KiCad board)
At the start: 2 copper layers, 186.4 x 104 mm, 61 parts, among them J1 PWR IN 12V, J2 LINE IN, J3 SPEAKER 4R, Q1 IRF540N, Q2 IRF540N, Q3 IRF540N, Q4 IRF540N, U1 TL074, U2 LM311, U3 LM311, U4 LM311, U5 CD4049UBE, U6 HIP4082IPZ

Commit message: Class D: the autoplace and routing experiments, hand and machine
Both placements of the same board, each carried through refine and route, plus
the DRC dump and the Freerouting session files.

Measured on these files with the same router pass and the same cnc clearance
profile: the hand placement needs 17 hand-soldered links against the machine
placement's 26, while beating it on normalised wirelength as well, 0.1053 to
0.1184. Worth keeping the pair around -- one netlist with two placements is the
only way to compare a placer against anything.
Parts:
- moved TP1 26.3 mm to (94.8, 74.2)
- moved RV1 26.2 mm to (78.2, 63.8), turned to 90 degrees
- moved C8 23.8 mm to (102.7, 84.8)
- moved TP2 23.8 mm to (87.3, 102.9)
- moved R8 23.5 mm to (122.1, 74.4)
- moved R9 23.1 mm to (126.8, 52.0)
- moved C12 23.0 mm to (104.2, 65.1)
- moved C4 23.0 mm to (180.4, 114.1)
- moved C5 23.0 mm to (153.4, 105.8)
- moved C6 23.0 mm to (141.2, 82.7)
- moved C7 23.0 mm to (120.8, 36.3)
- moved D3 23.0 mm to (134.0, 87.8)
- moved L2 23.0 mm to (165.5, 88.1)
- moved Q3 23.0 mm to (165.9, 102.1)
- moved R1 23.0 mm to (91.5, 53.3)
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Routing:
- net +12V: track 0.00 -> 324.1 mm
- net /AUDIO_N: track 0.00 -> 197.8 mm
- net /SQ: track 0.00 -> 124.0 mm
- net /G_BL: track 0.00 -> 113.4 mm
- net /TRI: track 0.00 -> 99.5 mm
- net /SW_B: track 0.00 -> 98.1 mm
- net /SW_A: track 0.00 -> 87.9 mm
- net /A_LO: track 0.00 -> 77.6 mm
- net /OUT_P: track 0.00 -> 77.1 mm
- net /PWM_A: track 0.00 -> 74.1 mm
- net /AUDIO_P: track 0.00 -> 65.1 mm
- net Net-(U1A-+): track 0.00 -> 47.9 mm
- net /A_HI: track 0.00 -> 41.2 mm
- net Net-(U1B--): track 0.00 -> 39.3 mm
- net /VGND: track 0.00 -> 35.8 mm
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- added copper zone on B.Cu, net GND
- removed copper zone on F.Cu, net GND
Other:
- board size 186.4 x 104 mm -> 190.5 x 104 mm
- board text added: "SRM-20 stroke 203.2 x 152.4"
- board text added: "via blank 190 x 140"
