File: Projects/Vinyl ADC/hardware/kicad/channel_l/vinyl_adc_channel_l.kicad_sch (KiCad schematic)
At the start: 39 parts, among them J20 LINE IN L, J21 Q SEL, J7 2x8 BUS, U20 TL072, U21 LM311, U22 TL072, U23 74HC74, U24 74HC04

Commit message: Vinyl ADC: channel artwork finished, and its production set
VREF_N to J7 pin 6 is routed -- the one link FreeRouting would not close
at 30 or 100 passes with the whole top layer free. The channel board is
now 26/26 nets in one piece, both oracles agreeing at 0 unconnected, 0
vias, 0 stranded pads.

Its ground pour was in ten pieces: the GND zone had island removal set to
Never, leaving nine floating fragments of 1.2 to 12.9 mm2, none carrying
a pad, all reported as isolated_copper. Set to Always and refilled. Pour
is one piece, those nine DRC violations are gone, and nothing depended on
them -- zero stranded pads before and after. DRC now reports nothing but
thirteen silk_overlap.

The schematic moved on the page by a uniform +19.05, +57.15 mm. Netlist
unchanged: check_split still accounts for all 92 nets and 377 nodes, and
check_fixture still passes.

One thing worth knowing that is NOT in the acceptance bar: cutspan reads
1.141 board diagonals against 0.725 for the automated route. The ground
return detours 161 mm further than the straight line and the worst point
is J7 pin 1, the bus GND pin. Not a fault, does not block the mill, but
this artwork is cut twice and feeds a modulator whose noise floor is
ground-dependent.

The production set is versioned here rather than ignored, against the
policy in production/.gitignore, because it has to be reachable from the
CAM machine and that machine has no KiCad. It is committed alongside the
exact board it came from, so it is not the stale set that policy exists
to prevent. Regenerate rather than edit it.

export_production.ps1 could not write the gerbers: it passes
-o "$OutDir\gerbers\", and the trailing backslash before the closing
quote is read as an escaped quote, so the path ran on and came back as
personal-projects\ADC\... -- kicad-cli then reported the board missing.
Invisible unless the path has a space in it, and "Vinyl ADC" has one. The
DXF steps pass a full filename and were fine. Gerbers and drill exported
by h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
Other:
- moved on the sheet: C20, C21, C22, C23, C24, C25, C26, C27, C28, C29, C30, C31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
