File: Projects/Vinyl ADC/hardware/kicad/power/vinyl_adc_power.kicad_pcb (KiCad board)
At the start: 2 copper layers, 100 x 100 mm, 22 parts, among them J3 2x8 BUS, U1 74HC244, U2 TL072

Commit message: Vinyl ADC: the digital and power layouts as fabricated
The two boards milled on 2026-09-03, side by side on one sheet. Editor
history folders are ignored from here on.
Parts:
- added WL1A: -5V, WireLink_TH, F.Cu at (86.0, 37.5)
- added WL1B: -5V, WireLink_TH, F.Cu at (54.0, 28.5)
Routing:
- net +5V: track 272.2 -> 186.8 mm
- net -5V: track 53.7 -> 88.1 mm
- net VREF_N: track 82.9 -> 77.5 mm
- net Net-(U1-1Y0): track 100.8 -> 103.1 mm
- net Net-(U2A-+): track 13.7 -> 15.6 mm
