File: esp32-node/esp32node/wip_route/esp32node_wip.kicad_pcb (KiCad board)
At the start: 2 copper layers, 63 x 60.8 mm, 32 parts, among them J1 USB-C, J2 GPIO L, J3 GPIO R, J4 I2C, J5 1-Wire, Q1 S8050, Q2 S8050, SW1 RESET, SW2 BOOT, U1 ESP32-WROOM-32, U2 AMS1117-3.3, U3 CH340C

Commit message: ESP32 boards: link footprints to their schematic symbols
Script-built boards had no footprint library IDs and no symbol paths, so
KiCad saw every part as unrelated to the schematic (17/17 and 32/32
footprint_symbol_mismatch in schematic-parity DRC). relink_pcb.py sets
LIB_ID, symbol path and sheet fields from the netlist without touching
placement or copper; bootstrap_pcb.py now does it when building. Both
boards pass schematic parity with 0 mismatches.
Parts:
- C1, C2, C3, C4, C5, C6, C7: footprint C_0805_2012Metric -> Capacitor_SMD:C_0805_2012Metric
- D1, D2: footprint LED_0805_2012Metric -> LED_SMD:LED_0805_2012Metric
- J1: footprint USB_C_Receptacle_GCT_USB4105-xx-A_16P_TopMnt_Horizontal -> Connector_USB:USB_C_Receptacle_GCT_USB4105-xx-A_16P_TopMnt_Horizontal
- J2, J3: footprint PinHeader_1x16_P2.54mm_Vertical -> Connector_PinHeader_2.54mm:PinHeader_1x16_P2.54mm_Vertical
- J4: footprint PinHeader_1x04_P2.54mm_Vertical -> Connector_PinHeader_2.54mm:PinHeader_1x04_P2.54mm_Vertical
- J5: footprint PinHeader_1x03_P2.54mm_Vertical -> Connector_PinHeader_2.54mm:PinHeader_1x03_P2.54mm_Vertical
- Q1, Q2: footprint SOT-23 -> Package_TO_SOT_SMD:SOT-23
- R1, R10, R11, R2, R3, R4, R5, R6, R7, R8, R9: footprint R_0805_2012Metric -> Resistor_SMD:R_0805_2012Metric
- SW1, SW2: footprint SW_SPST_PTS645Sx43SMTR92 -> Button_Switch_SMD:SW_SPST_PTS645Sx43SMTR92
- U1: footprint ESP32-WROOM-32_NoVias -> esp32node:ESP32-WROOM-32_NoVias
- U2: footprint SOT-223-3_TabPin2 -> Package_TO_SOT_SMD:SOT-223-3_TabPin2
- U3: footprint SOIC-16_3.9x9.9mm_P1.27mm -> Package_SO:SOIC-16_3.9x9.9mm_P1.27mm
Changed lines of the file:
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@@
 		)
 	)
-	(footprint "PinHeader_1x16_P2.54mm_Vertical"
+	(footprint "Connector_PinHeader_2.54mm:PinHeader_1x16_P2.54mm_Vertical"
 		(layer "F.Cu")
 		(at 126 93)
@@
 			)
 		)
+		(sheetname "esp32node")
+		(sheetfile "esp32node.kicad_sch")
 		(attr through_hole)
 		(duplicate_pad_numbers_are_jumpers no)
@@
 		)
 	)
-	(footprint "PinHeader_1x16_P2.54mm_Vertical"
+	(footprint "Connector_PinHeader_2.54mm:PinHeader_1x16_P2.54mm_Vertical"
 		(layer "F.Cu")
 		(at 174 93)
@@
 			)
 		)
+		(sheetname "esp32node")
+		(sheetfile "esp32node.kicad_sch")
 		(attr through_hole)
 		(duplicate_pad_numbers_are_jumpers no)
@@
 		)
 	)
-	(footprint "PinHeader_1x03_P2.54mm_Vertical"
+	(footprint "Connector_PinHeader_2.54mm:PinHeader_1x03_P2.54mm_Vertical"
 		(layer "F.Cu")
 		(at 138 127)
@@
 			)
 		)
+		(sheetname "esp32node")
+		(sheetfile "esp32node.kicad_sch")
 		(attr through_hole)
 		(duplicate_pad_numbers_are_jumpers no)
@@
 		)
 	)
-	(footprint "PinHeader_1x04_P2.54mm_Vertical"
+	(footprint "Connector_PinHeader_2.54mm:PinHeader_1x04_P2.54mm_Vertical"
 		(layer "F.Cu")
 		(at 119.8 144 90)
@@
 			)
 		)
+		(sheetname "esp32node")
+		(sheetfile "esp32node.kicad_sch")
 		(attr through_hole)
 		(duplicate_pad_numbers_are_jumpers no)
@@
 		)
 	)
-	(footprint "R_0805_2012Metric"
+	(footprint "Resistor_SMD:R_0805_2012Metric"
 		(layer "B.Cu")
 		(at 141.5 128 -90)
@@
 			)
 		)
+		(sheetname "esp32node")
+		(sheetfile "esp32node.kicad_sch")
 		(attr smd)
 		(duplicate_pad_numbers_are_jumpers no)
@@
 		)
 	)
-	(footprint "SW_SPST_PTS645Sx43SMTR92"
+	(footprint "Button_Switch_SMD:SW_SPST_PTS645Sx43SMTR92"
 		(layer "B.Cu")
 		(at 150 114.5 180)
@@
 			)
 		)
+		(sheetname "esp32node")
+		(sheetfile "esp32node.kicad_sch")
 		(attr smd)
 		(duplicate_pad_numbers_are_jumpers no)
@@
 		)
 	)
-	(footprint "C_0805_2012Metric"
+	(footprint "Capacitor_SMD:C_0805_2012Metric"
 		(layer "B.Cu")
 		(at 177.4 96 -90)
@@
 			)
 		)
+		(sheetname "esp32node")
+		(sheetfile "esp32node.kicad_sch")
 		(attr smd)
 		(duplicate_pad_numbers_are_jumpers no)
@@
 		)
 	)
-	(footprint "SOT-23"
+	(footprint "Package_TO_SOT_SMD:SOT-23"
 		(layer "B.Cu")
 		(at 139 121 180)
@@
 			)
 		)
+		(sheetname "esp32node")
+		(sheetfile "esp32node.kicad_sch")
 		(attr smd)
 		(duplicate_pad_numbers_are_jumpers no)
@@
 		)
 	)
-	(footprint "SW_SPST_PTS645Sx43SMTR92"
+	(footprint "Button_Switch_SMD:SW_SPST_PTS645Sx43SMTR92"
 		(layer "B.Cu")
 		(at 167 146.5 180)
@@
 			)
 		)
+		(sheetname "esp32node")
+		(sheetfile "esp32node.kicad_sch")
 		(attr smd)
 		(duplicate_pad_numbers_are_jumpers no)
@@
 		)
 	)
-	(footprint "R_0805_2012Metric"
+	(footprint "Resistor_SMD:R_0805_2012Metric"
 		(layer "B.Cu")
 		(at 124.88 147.8 -90)
@@
 			)
 		)
+		(sheetname "esp32node")
+		(sheetfile "esp32node.kicad_sch")
 		(attr smd)
 		(duplicate_pad_numbers_are_jumpers no)
@@
 		)
 	)
-	(footprint "R_0805_2012Metric"
+	(footprint "Resistor_SMD:R_0805_2012Metric"
 		(layer "B.Cu")
 		(at 134 126 -90)
@@
 			)
 		)
+		(sheetname "esp32node")
+		(sheetfile "esp32node.kicad_sch")
 		(attr smd)
 		(duplicate_pad_numbers_are_jumpers no)
@@
 		)
 	)
-	(footprint "R_0805_2012Metric"
+	(footprint "Resistor_SMD:R_0805_2012Metric"
 		(layer "B.Cu")
 		(at 143 121 -90)
@@
 			)
 		)
+		(sheetname "esp32node")
+		(sheetfile "esp32node.kicad_sch")
 		(attr smd)
 		(duplicate_pad_numbers_are_jumpers no)
@@
 		)
 	)
-	(footprint "R_0805_2012Metric"
+	(footprint "Resistor_SMD:R_0805_2012Metric"
 		(layer "B.Cu")
 		(at 177.4 123 -90)
@@
 			)
 		)
+		(sheetname "esp32node")
+		(sheetfile "esp32node.kicad_sch")
 		(attr smd)
 		(duplicate_pad_numbers_are_jumpers no)
@@
 		)
 	)
-	(footprint "LED_0805_2012Metric"
+	(footprint "LED_SMD:LED_0805_2012Metric"
 		(layer "B.Cu")
 		(at 177.4 143 -90)
@@
 			)
 		)
+		(sheetname "esp32node")
+		(sheetfile "esp32node.kicad_sch")
 		(attr smd)
 		(duplicate_pad_numbers_are_jumpers no)
@@
 		)
 	)
-	(footprint "C_0805_2012Metric"
+	(footprint "Capacitor_SMD:C_0805_2012Metric"
 		(layer "B.Cu")
 		(at 177.4 128 -90)
@@
 			)
 		)
+		(sheetname "esp32node")
+		(sheetfile "esp32node.kicad_sch")
 		(attr smd)
 		(duplicate_pad_numbers_are_jumpers no)
@@
 		)
 	)
-	(footprint "C_0805_2012Metric"
+	(footprint "Capacitor_SMD:C_0805_2012Metric"
 		(layer "B.Cu")
 		(at 137 139.5 180)
@@
 			)
 		)
+		(sheetname "esp32node")
+		(sheetfile "esp32node.kicad_sch")
 		(attr smd)
 		(duplicate_pad_numbers_are_jumpers no)
@@
 		)
 	)
-	(footprint "ESP32-WROOM-32_NoVias"
+	(footprint "esp32node:ESP32-WROOM-32_NoVias"
 		(layer "B.Cu")
 		(at 150 100 180)
@@
 			)
 		)
+		(sheetname "esp32node")
+		(sheetfile "esp32node.kicad_sch")
 		(attr smd)
 		(duplicate_pad_numbers_are_jumpers no)
@@
 		)
 	)
-	(footprint "USB_C_Receptacle_GCT_USB4105-xx-A_16P_TopMnt_Horizontal"
+	(footprint "Connector_USB:USB_C_Receptacle_GCT_USB4105-xx-A_16P_TopMnt_Horizontal"
 		(layer "B.Cu")
 		(at 150 147.1 180)
@@
 			)
 		)
+		(sheetname "esp32node")
+		(sheetfile "esp32node.kicad_sch")
 		(attr smd)
 		(duplicate_pad_numbers_are_jumpers no)
@@
 		)
 	)
-	(footprint "R_0805_2012Metric"
+	(footprint "Resistor_SMD:R_0805_2012Metric"
 		(layer "B.Cu")
 		(at 157.5 139 -90)
@@
 			)
 		)
+		(sheetname "esp32node")
+		(sheetfile "esp32node.kicad_sch")
 		(attr smd)
 		(duplicate_pad_numbers_are_jumpers no)
@@
 		)
 	)
-	(footprint "SOT-23"
+	(footprint "Package_TO_SOT_SMD:SOT-23"
 		(layer "B.Cu")
 		(at 164.5 124 180)
@@
 			)
 		)
+		(sheetname "esp32node")
+		(sheetfile "esp32node.kicad_sch")
 		(attr smd)
 		(duplicate_pad_numbers_are_jumpers no)
@@
 		)
 	)
-	(footprint "SOIC-16_3.9x9.9mm_P1.27mm"
+	(footprint "Package_SO:SOIC-16_3.9x9.9mm_P1.27mm"
 		(layer "B.Cu")
 		(at 152 124 90)
@@
 			)
 		)
+		(sheetname "esp32node")
+		(sheetfile "esp32node.kicad_sch")
 		(attr smd)
 		(duplicate_pad_numbers_are_jumpers no)
@@
 		)
 	)
-	(footprint "LED_0805_2012Metric"
+	(footprint "LED_SMD:LED_0805_2012Metric"
 		(layer "B.Cu")
 		(at 134 130 -90)
@@
 			)
 		)
+		(sheetname "esp32node")
+		(sheetfile "esp32node.kicad_sch")
 		(attr smd)
 		(duplicate_pad_numbers_are_jumpers no)
@@
 		)
 	)
-	(footprint "R_0805_2012Metric"
+	(footprint "Resistor_SMD:R_0805_2012Metric"
 		(layer "B.Cu")
 		(at 122.34 147.8 -90)
@@
 			)
 		)
+		(sheetname "esp32node")
+		(sheetfile "esp32node.kicad_sch")
 		(attr smd)
 		(duplicate_pad_numbers_are_jumpers no)
@@
 		)
 	)
-	(footprint "R_0805_2012Metric"
+	(footprint "Resistor_SMD:R_0805_2012Metric"
 		(layer "B.Cu")
 		(at 160.5 124 -90)
@@
 			)
 		)
+		(sheetname "esp32node")
+		(sheetfile "esp32node.kicad_sch")
 		(attr smd)
 		(duplicate_pad_numbers_are_jumpers no)
@@
 		)
 	)
-	(footprint "SOT-223-3_TabPin2"
+	(footprint "Package_TO_SOT_SMD:SOT-223-3_TabPin2"
 		(layer "B.Cu")
 		(at 137 146 180)
@@
 			)
 		)
+		(sheetname "esp32node")
+		(sheetfile "esp32node.kicad_sch")
 		(attr smd)
 		(duplicate_pad_numbers_are_jumpers no)
@@
 		)
 	)
-	(footprint "R_0805_2012Metric"
+	(footprint "Resistor_SMD:R_0805_2012Metric"
 		(layer "B.Cu")
 		(at 158 112.5 -90)
@@
 			)
 		)
+		(sheetname "esp32node")
+		(sheetfile "esp32node.kicad_sch")
 		(attr smd)
 		(duplicate_pad_numbers_are_jumpers no)
@@
 		)
 	)
-	(footprint "C_0805_2012Metric"
+	(footprint "Capacitor_SMD:C_0805_2012Metric"
 		(layer "B.Cu")
 		(at 159 119 -90)
@@
 			)
 		)
+		(sheetname "esp32node")
+		(sheetfile "esp32node.kicad_sch")
 		(attr smd)
 		(duplicate_pad_numbers_are_jumpers no)
@@
 		)
 	)
-	(footprint "R_0805_2012Metric"
+	(footprint "Resistor_SMD:R_0805_2012Metric"
 		(layer "B.Cu")
 		(at 142.5 139 -90)
@@
 			)
 		)
+		(sheetname "esp32node")
+		(sheetfile "esp32node.kicad_sch")
 		(attr smd)
 		(duplicate_pad_numbers_are_jumpers no)
@@
 		)
 	)
-	(footprint "C_0805_2012Metric"
+	(footprint "Capacitor_SMD:C_0805_2012Metric"
 		(layer "B.Cu")
 		(at 130 147 -90)
@@
 			)
 		)
+		(sheetname "esp32node")
+		(sheetfile "esp32node.kicad_sch")
 		(attr smd)
 		(duplicate_pad_numbers_are_jumpers no)
@@
 		)
 	)
-	(footprint "R_0805_2012Metric"
+	(footprint "Resistor_SMD:R_0805_2012Metric"
 		(layer "B.Cu")
 		(at 177.4 138.5 -90)
@@
 			)
 		)
+		(sheetname "esp32node")
+		(sheetfile "esp32node.kicad_sch")
 		(attr smd)
 		(duplicate_pad_numbers_are_jumpers no)
@@
 		)
 	)
-	(footprint "C_0805_2012Metric"
+	(footprint "Capacitor_SMD:C_0805_2012Metric"
 		(layer "B.Cu")
 		(at 162 93 -90)
@@
 			)
 		)
+		(sheetname "esp32node")
+		(sheetfile "esp32node.kicad_sch")
 		(attr smd)
 		(duplicate_pad_numbers_are_jumpers no)
@@
 		)
 	)
-	(footprint "C_0805_2012Metric"
+	(footprint "Capacitor_SMD:C_0805_2012Metric"
 		(layer "B.Cu")
 		(at 156.5 130.5 -90)
@@
 			)
 		)
+		(sheetname "esp32node")
+		(sheetfile "esp32node.kicad_sch")
 		(attr smd)
 		(duplicate_pad_numbers_are_jumpers no)
