File: esp32-solder-test/esp32solder.placed.kicad_pcb (KiCad board)
At the start: 2 copper layers, 54 x 45.8 mm, 17 parts, among them J1 UART / 5V, SW1 RESET, SW2 BOOT, U1 ESP32-WROOM-32, U2 LM317T

Commit message: ESP32 boards: link footprints to their schematic symbols
Script-built boards had no footprint library IDs and no symbol paths, so
KiCad saw every part as unrelated to the schematic (17/17 and 32/32
footprint_symbol_mismatch in schematic-parity DRC). relink_pcb.py sets
LIB_ID, symbol path and sheet fields from the netlist without touching
placement or copper; bootstrap_pcb.py now does it when building. Both
boards pass schematic parity with 0 mismatches.
Parts:
- C1, C2, C4: footprint CP_Radial_D5.0mm_P2.00mm -> Capacitor_THT:CP_Radial_D5.0mm_P2.00mm
- C3: footprint C_Disc_D3.0mm_W1.6mm_P2.50mm -> Capacitor_THT:C_Disc_D3.0mm_W1.6mm_P2.50mm
- D1, D2: footprint LED_D3.0mm -> LED_THT:LED_D3.0mm
- J1: footprint PinHeader_1x04_P2.54mm_Vertical -> Connector_PinHeader_2.54mm:PinHeader_1x04_P2.54mm_Vertical
- R1, R2, R3, R4, R5, R6: footprint R_Axial_DIN0207_L6.3mm_D2.5mm_P10.16mm_Horizontal -> Resistor_THT:R_Axial_DIN0207_L6.3mm_D2.5mm_P10.16mm_Horizontal
- SW1, SW2: footprint SW_PUSH_6mm -> Button_Switch_THT:SW_PUSH_6mm
- U1: footprint ESP32-WROOM-32_NoVias -> esp32solder:ESP32-WROOM-32_NoVias
- U2: footprint TO-220-3_Vertical -> Package_TO_SOT_THT:TO-220-3_Vertical
Changed lines of the file:
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@@
 		)
 	)
-	(footprint "R_Axial_DIN0207_L6.3mm_D2.5mm_P10.16mm_Horizontal"
+	(footprint "Resistor_THT:R_Axial_DIN0207_L6.3mm_D2.5mm_P10.16mm_Horizontal"
 		(layer "F.Cu")
 		(at 174.16 100.5 180)
@@
 			)
 		)
+		(sheetname "esp32solder")
+		(sheetfile "esp32solder.kicad_sch")
 		(attr through_hole)
 		(duplicate_pad_numbers_are_jumpers no)
@@
 		)
 	)
-	(footprint "R_Axial_DIN0207_L6.3mm_D2.5mm_P10.16mm_Horizontal"
+	(footprint "Resistor_THT:R_Axial_DIN0207_L6.3mm_D2.5mm_P10.16mm_Horizontal"
 		(layer "F.Cu")
 		(at 141 122.66 90)
@@
 			)
 		)
+		(sheetname "esp32solder")
+		(sheetfile "esp32solder.kicad_sch")
 		(attr through_hole)
 		(duplicate_pad_numbers_are_jumpers no)
@@
 		)
 	)
-	(footprint "CP_Radial_D5.0mm_P2.00mm"
+	(footprint "Capacitor_THT:CP_Radial_D5.0mm_P2.00mm"
 		(layer "F.Cu")
 		(at 135.54 125.5)
@@
 			)
 		)
+		(sheetname "esp32solder")
+		(sheetfile "esp32solder.kicad_sch")
 		(attr through_hole)
 		(duplicate_pad_numbers_are_jumpers no)
@@
 		)
 	)
-	(footprint "TO-220-3_Vertical"
+	(footprint "Package_TO_SOT_THT:TO-220-3_Vertical"
 		(layer "F.Cu")
 		(at 138.08 131.5 180)
@@
 			)
 		)
+		(sheetname "esp32solder")
+		(sheetfile "esp32solder.kicad_sch")
 		(attr through_hole)
 		(duplicate_pad_numbers_are_jumpers no)
@@
 		)
 	)
-	(footprint "CP_Radial_D5.0mm_P2.00mm"
+	(footprint "Capacitor_THT:CP_Radial_D5.0mm_P2.00mm"
 		(layer "F.Cu")
 		(at 164 105)
@@
 			)
 		)
+		(sheetname "esp32solder")
+		(sheetfile "esp32solder.kicad_sch")
 		(attr through_hole)
 		(duplicate_pad_numbers_are_jumpers no)
@@
 		)
 	)
-	(footprint "CP_Radial_D5.0mm_P2.00mm"
+	(footprint "Capacitor_THT:CP_Radial_D5.0mm_P2.00mm"
 		(layer "F.Cu")
 		(at 128.5 127)
@@
 			)
 		)
+		(sheetname "esp32solder")
+		(sheetfile "esp32solder.kicad_sch")
 		(attr through_hole)
 		(duplicate_pad_numbers_are_jumpers no)
@@
 		)
 	)
-	(footprint "LED_D3.0mm"
+	(footprint "LED_THT:LED_D3.0mm"
 		(layer "F.Cu")
 		(at 177 129.04 90)
@@
 			)
 		)
+		(sheetname "esp32solder")
+		(sheetfile "esp32solder.kicad_sch")
 		(attr through_hole)
 		(duplicate_pad_numbers_are_jumpers no)
@@
 		)
 	)
-	(footprint "R_Axial_DIN0207_L6.3mm_D2.5mm_P10.16mm_Horizontal"
+	(footprint "Resistor_THT:R_Axial_DIN0207_L6.3mm_D2.5mm_P10.16mm_Horizontal"
 		(layer "F.Cu")
 		(at 142 131.5)
@@
 			)
 		)
+		(sheetname "esp32solder")
+		(sheetfile "esp32solder.kicad_sch")
 		(attr through_hole)
 		(duplicate_pad_numbers_are_jumpers no)
@@
 		)
 	)
-	(footprint "SW_PUSH_6mm"
+	(footprint "Button_Switch_THT:SW_PUSH_6mm"
 		(layer "F.Cu")
 		(at 169.5 104.5)
@@
 			)
 		)
+		(sheetname "esp32solder")
+		(sheetfile "esp32solder.kicad_sch")
 		(attr through_hole)
 		(duplicate_pad_numbers_are_jumpers no)
@@
 		)
 	)
-	(footprint "SW_PUSH_6mm"
+	(footprint "Button_Switch_THT:SW_PUSH_6mm"
 		(layer "F.Cu")
 		(at 129.5 112)
@@
 			)
 		)
+		(sheetname "esp32solder")
+		(sheetfile "esp32solder.kicad_sch")
 		(attr through_hole)
 		(duplicate_pad_numbers_are_jumpers no)
@@
 		)
 	)
-	(footprint "R_Axial_DIN0207_L6.3mm_D2.5mm_P10.16mm_Horizontal"
+	(footprint "Resistor_THT:R_Axial_DIN0207_L6.3mm_D2.5mm_P10.16mm_Horizontal"
 		(layer "F.Cu")
 		(at 144.28 112.5 -90)
@@
 			)
 		)
+		(sheetname "esp32solder")
+		(sheetfile "esp32solder.kicad_sch")
 		(attr through_hole)
 		(duplicate_pad_numbers_are_jumpers no)
@@
 		)
 	)
-	(footprint "PinHeader_1x04_P2.54mm_Vertical"
+	(footprint "Connector_PinHeader_2.54mm:PinHeader_1x04_P2.54mm_Vertical"
 		(layer "F.Cu")
 		(at 131.5 93.56)
@@
 			)
 		)
+		(sheetname "esp32solder")
+		(sheetfile "esp32solder.kicad_sch")
 		(attr through_hole)
 		(duplicate_pad_numbers_are_jumpers no)
@@
 		)
 	)
-	(footprint "C_Disc_D3.0mm_W1.6mm_P2.50mm"
+	(footprint "Capacitor_THT:C_Disc_D3.0mm_W1.6mm_P2.50mm"
 		(layer "F.Cu")
 		(at 162.5 93.02 -90)
@@
 			)
 		)
+		(sheetname "esp32solder")
+		(sheetfile "esp32solder.kicad_sch")
 		(attr through_hole)
 		(duplicate_pad_numbers_are_jumpers no)
@@
 		)
 	)
-	(footprint "LED_D3.0mm"
+	(footprint "LED_THT:LED_D3.0mm"
 		(layer "F.Cu")
 		(at 149.82 122.66 180)
@@
 			)
 		)
+		(sheetname "esp32solder")
+		(sheetfile "esp32solder.kicad_sch")
 		(attr through_hole)
 		(duplicate_pad_numbers_are_jumpers no)
@@
 		)
 	)
-	(footprint "R_Axial_DIN0207_L6.3mm_D2.5mm_P10.16mm_Horizontal"
+	(footprint "Resistor_THT:R_Axial_DIN0207_L6.3mm_D2.5mm_P10.16mm_Horizontal"
 		(layer "F.Cu")
 		(at 155.5 131.5 90)
@@
 			)
 		)
+		(sheetname "esp32solder")
+		(sheetfile "esp32solder.kicad_sch")
 		(attr through_hole)
 		(duplicate_pad_numbers_are_jumpers no)
@@
 		)
 	)
-	(footprint "R_Axial_DIN0207_L6.3mm_D2.5mm_P10.16mm_Horizontal"
+	(footprint "Resistor_THT:R_Axial_DIN0207_L6.3mm_D2.5mm_P10.16mm_Horizontal"
 		(layer "F.Cu")
 		(at 177 113 -90)
@@
 			)
 		)
+		(sheetname "esp32solder")
+		(sheetfile "esp32solder.kicad_sch")
 		(attr through_hole)
 		(duplicate_pad_numbers_are_jumpers no)
@@
 		)
 	)
-	(footprint "ESP32-WROOM-32_NoVias"
+	(footprint "esp32solder:ESP32-WROOM-32_NoVias"
 		(layer "B.Cu")
 		(at 150 100 180)
@@
 			)
 		)
+		(sheetname "esp32solder")
+		(sheetfile "esp32solder.kicad_sch")
 		(attr smd)
 		(duplicate_pad_numbers_are_jumpers no)
